File: Placa/pcb bobinadora.sch (EAGLE design)
At the start: 20 parts, among them IC1 PIC16F84AP, Q1 4 MhZ, SW1 MOMENTARY, SW2 MOMENTARY, SW3 MOMENTARY, X1 87758-3416

Commit message: final
Parts:
- removed V1: 9VBATTERY, gm-supply:9VBATTERY
- removed X1: 87758-3416, con-molex:87758-3416
- added +9V1: +9V(T), gm-supply:+9V(T)
- added JP2: (no value), pinhead:PINHD-1X16
Connections:
- removed net N$18: C4.+, REG1.VI, V1.+
- new net N$17: JP2.1, JP2.5
- net GND: no longer V1.-, X1-18.S
- net N$1: now also JP2.11; no longer X1-28.S
- net N$2: now also JP2.12; no longer X1-30.S
- net N$3: now also JP2.13; no longer X1-32.S
- net N$4: now also JP2.14; no longer X1-34.S
- net N$5: now also JP2.4; no longer X1-16.S
- net N$6: now also JP2.6; no longer X1-20.S
- net PWR: now also +9V1.+9V, C4.+, JP2.2, REG1.VI
